File: Display.kicad_sch (KiCad schematic)
At the start: 27 parts, among them J2 TFT_LCD, U3 MT9284, U5 TPS61169

Commit message: Move to Kicad V.9. Added Pinout for CubeIDE
Changed lines of the file:
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@@
 (kicad_sch
-	(version 20231120)
+	(version 20250114)
 	(generator "eeschema")
-	(generator_version "8.0")
+	(generator_version "9.0")
 	(paper "A4")
+	(text "100mA"
+		(exclude_from_sim no)
+		(at 111.76 159.258 0)
+		(effects
+			(font
+				(size 1.27 1.27)
+			)
+		)
+	)
+	(text "50mA"
+		(exclude_from_sim no)
+		(at 103.124 159.258 0)
+		(effects
+			(font
+				(size 1.27 1.27)
+			)
+		)
+	)
+	(text "25mA"
+		(exclude_from_sim no)
+		(at 93.98 159.258 0)
+		(effects
+			(font
+				(size 1.27 1.27)
+			)
+		)
+	)
+	(text "Please check Adafruit Qualia ESP32-S3 for TTL RGB-666 Displays"
+		(exclude_from_sim no)
+		(at 49.784 154.94 0)
+		(effects
+			(font
+				(size 1.27 1.27)
+			)
+		)
+	)
 	(junction
 		(at 52.07 119.38)
@@
 		)
 	)
-	(text "100mA"
-		(exclude_from_sim no)
-		(at 111.76 159.258 0)
-		(effects
-			(font
-				(size 1.27 1.27)
-			)
-		)
-	)
-	(text "50mA"
-		(exclude_from_sim no)
-		(at 103.124 159.258 0)
-		(effects
-			(font
-				(size 1.27 1.27)
-			)
-		)
-	)
-	(text "25mA"
-		(exclude_from_sim no)
-		(at 93.98 159.258 0)
-		(effects
-			(font
-				(size 1.27 1.27)
-			)
-		)
-	)
-	(text "Please check Adafruit Qualia ESP32-S3 for TTL RGB-666 Displays"
-		(exclude_from_sim no)
-		(at 49.784 154.94 0)
-		(effects
-			(font
-				(size 1.27 1.27)
-			)
-		)
-	)
 	(label "LED_K"
 		(at 94.615 204.47 180)
-		(fields_autoplaced yes)
 		(effects
 			(font
@@
 	(label "LCD_B5"
 		(at 194.31 76.2 0)
-		(fields_autoplaced yes)
 		(effects
 			(font
@@
 	(label "LCD_TP_INT"
 		(at 194.31 116.84 0)
-		(fields_autoplaced yes)
 		(effects
 			(font
@@
 	(label "LCD_SPI_CS"
 		(at 194.31 55.88 0)
-		(fields_autoplaced yes)
 		(effects
 			(font
@@
 	(label "LCD_G7"
 		(at 194.31 96.52 0)
-		(fields_autoplaced yes)
 		(effects
 			(font
@@
 	(label "LCD_BLK"
 		(at 57.15 48.26 0)
-		(fields_autoplaced yes)
 		(effects
 			(font
@@
 	(label "LCD_G5"
 		(at 194.31 91.44 0)
-		(fields_autoplaced yes)
 		(effects
 			(font
@@
 	(label "LCD_B3"
 		(at 194.31 71.12 0)
-		(fields_autoplaced yes)
 		(effects
 			(font
@@
 	(label "LED_A"
 		(at 195.58 30.48 0)
-		(fields_autoplaced yes)
 		(effects
 			(font
@@
 	(label "LCD_B6"
 		(at 194.31 78.74 0)
-		(fields_autoplaced yes)
 		(effects
 			(font
@@
 	(label "LED_K"
 		(at 121.92 133.35 180)
-		(fields_autoplaced yes)
 		(effects
 			(font
@@
 	(label "LED_K"
 		(at 195.58 33.02 0)
-		(fields_autoplaced yes)
 		(effects
 			(font
@@
 	(label "VSYNC"
 		(at 194.31 63.5 0)
-		(fields_autoplaced yes)
 		(effects
 			(font
@@
 	(label "LCD_TP_SCL"
 		(at 173.99 121.92 180)
-		(fields_autoplaced yes)
 		(effects
 			(font
@@
 	(label "HSYNC"
 		(at 194.31 66.04 0)
-		(fields_autoplaced yes)
 		(effects
 			(font
@@
 	(label "LCD_DE"
 		(at 194.31 60.96 0)
-		(fields_autoplaced yes)
 		(effects
 			(font
@@
 	(label "LCD_G6"
 		(at 194.31 93.98 0)
-		(fields_autoplaced yes)
 		(effects
 			(font
@@
 	(label "LCD_TP_SDA"
 		(at 194.31 119.38 0)
-		(fields_autoplaced yes)
 		(effects
 			(font
@@
 	(label "LCD_TP_SDA"
 		(at 173.99 119.38 180)
-		(fields_autoplaced yes)
 		(effects
 			(font
@@
 	(label "LCD_G4"
 		(at 194.31 88.9 0)
-		(fields_autoplaced yes)
 		(effects
 			(font
@@
 	(label "LCD_G3"
 		(at 194.31 86.36 0)
-		(fields_autoplaced yes)
 		(effects
 			(font
@@
 	(label "LCD_G2"
 		(at 194.31 83.82 0)
-		(fields_autoplaced yes)
 		(effects
 			(font
@@
 	(label "LCD_CLK"
 		(at 194.31 58.42 0)
-		(fields_autoplaced yes)
 		(effects
 			(font
@@
 	(label "LCD_TP_SCL"
 		(at 194.31 121.92 0)
-		(fields_autoplaced yes)
 		(effects
 			(font
@@
 	(label "LED_A"
 		(at 107.95 114.3 180)
-		(fields_autoplaced yes)
 		(effects
 			(font
@@
 	(label "LCD_BLK"
 		(at 43.18 130.81 0)
-		(fields_autoplaced yes)
 		(effects
 			(font
@@
 	(label "LCD_SPI_DAT"
 		(at 194.31 50.8 0)
-		(fields_autoplaced yes)
 		(effects
 			(font
@@
 	(label "LCD_RESET"
 		(at 195.58 43.18 0)
-		(fields_autoplaced yes)
 		(effects
 			(font
@@
 	(label "LCD_TP_RST"
 		(at 194.31 124.46 0)
-		(fields_autoplaced yes)
 		(effects
 			(font
@@
 	(label "LCD_B7"
 		(at 194.31 81.28 0)
-		(fields_autoplaced yes)
 		(effects
 			(font
@@
 	(label "LCD_R3"
 		(at 194.31 101.6 0)
-		(fields_autoplaced yes)
 		(effects
 			(font
@@
 	(label "LED_K"
 		(at 135.255 48.26 180)
-		(fields_autoplaced yes)
 		(effects
 			(font
@@
 	(label "LCD_R7"
 		(at 194.31 111.76 0)
-		(fields_autoplaced yes)
 		(effects
 			(font
@@
 	(label "LED_A"
 		(at 135.255 43.18 180)
-		(fields_autoplaced yes)
 		(effects
 			(font
@@
 	(label "LCD_B4"
 		(at 194.31 73.66 0)
-		(fields_autoplaced yes)
 		(effects
 			(font
@@
 	(label "LCD_R5"
 		(at 194.31 106.68 0)
-		(fields_autoplaced yes)
 		(effects
 			(font
@@
 	(label "LCD_SPI_CLK"
 		(at 194.31 53.34 0)
-		(fields_autoplaced yes)
 		(effects
 			(font
@@
 	(label "LCD_R6"
 		(at 194.31 109.22 0)
-		(fields_autoplaced yes)
 		(effects
 			(font
@@
 	(label "LCD_R4"
 		(at 194.31 104.14 0)
-		(fields_autoplaced yes)
 		(effects
 			(font
@@
 		(shape input)
 		(at 194.31 58.42 180)
-		(fields_autoplaced yes)
 		(effects
 			(font
@@
 		(shape input)
 		(at 43.18 130.81 180)
-		(fields_autoplaced yes)
 		(effects
 			(font
@@
 		(shape bidirectional)
 		(at 194.31 119.38 180)
-		(fields_autoplaced yes)
 		(effects
 			(font
@@
 		(shape output)
 		(at 194.31 116.84 180)
-		(fields_autoplaced yes)
 		(effects
 			(font
@@
 		(shape input)
 		(at 194.31 60.96 180)
-		(fields_autoplaced yes)
 		(effects
 			(font
@@
 		(shape input)
 		(at 194.31 55.88 180)
-		(fields_autoplaced yes)
 		(effects
 			(font
@@
 		(shape input)
 		(at 194.31 124.46 180)
-		(fields_autoplaced yes)
 		(effects
 			(font
@@
 		(shape input)
 		(at 168.91 96.52 180)
-		(fields_autoplaced yes)
 		(effects
 			(font
@@
 		(shape input)
 		(at 194.31 53.34 180)
-		(fields_autoplaced yes)
 		(effects
 			(font
@@
 		(shape input)
 		(at 170.18 78.74 180)
-		(fields_autoplaced yes)
 		(effects
 			(font
@@
 		(shape input)
 		(at 194.31 121.92 180)
-		(fields_autoplaced yes)
 		(effects
 			(font
@@
 		(shape bidirectional)
 		(at 194.31 50.8 180)
-		(fields_autoplaced yes)
 		(effects
 			(font
@@
 		(shape input)
 		(at 195.58 43.18 180)
-		(fields_autoplaced yes)
 		(effects
 			(font
@@
 		(shape input)
 		(at 194.31 66.04 180)
-		(fields_autoplaced yes)
 		(effects
 			(font
@@
 		(shape input)
 		(at 173.99 66.04 180)
-		(fields_autoplaced yes)
 		(effects
 			(font
@@
 		(shape input)
 		(at 57.15 48.26 180)
-		(fields_autoplaced yes)
 		(effects
 			(font
@@
 		(shape input)
 		(at 194.31 63.5 180)
-		(fields_autoplaced yes)
-		(effects
-			(font
+		(effects
+			(font
