File: MAX98357.kicad_sch (KiCad schematic)
At the start: 6 parts, among them J8 SPKR, U6 MAX98357AETE_

Commit message: First release H743 version
Parts:
- R15: now not fitted; now left out of the parts list
- R16: value NC -> 100K; JLCPCB Part # (none) -> C60491
Changed lines of the file:
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@@
 			)
 		)
-		(property "Value" "NC"
+		(property "Value" "100K"
 			(at 69.85 97.7899 0)
 			(effects
@@
 			)
 		)
-		(property "JLCPCB Part #" ""
+		(property "JLCPCB Part #" "C60491"
 			(at 67.31 96.52 0)
 			(effects
@@
 		(unit 1)
 		(exclude_from_sim no)
-		(in_bom yes)
+		(in_bom no)
 		(on_board yes)
-		(dnp no)
+		(dnp yes)
 		(fields_autoplaced yes)
 		(property "Reference" "R15"
