File: STM32H743IIK6.kicad_sch (KiCad schematic)
At the start: 58 parts, among them J4 USB-C, J6 BAT, SW1 SW_Push, SW2 SW_Push, SW3 SW_Push, SW4 SW_Push, U10 STM32H743ZITx, U4 STM32H723ZGTx, U8 TLV75733PDBV, Y1 25MHz, Y2 32.768KHz

Commit message: LTDC route almost finished
Parts:
- removed U4: STM32H723ZGTx, Package_QFP:LQFP-144_20x20mm_P0.5mm, symbol MCU_ST_STM32H7:STM32H723ZGTx
Connections:
- net LCD_BLK: now also U10.43 (PA7)
- net LCD_RESET: now also U10.3 (PE4)
- net LCS_SPI_CLK: now also U10.1 (PE2)
- net LCS_SPI_CS: now also U10.2 (PE3)
- net LCS_SPI_DAT: now also U10.5 (PE6)
- net LTDC_B3: now also U10.126 (PG11)
- net LTDC_B4: now also U10.102 (PA10)
- net LTDC_B5: now also U10.37 (PA3)
- net LTDC_B6: now also U10.139 (PB8)
- net LTDC_B7: now also U10.140 (PB9)
- net LTDC_CLK: now also U10.92 (PG7)
- net LTDC_DE: now also U10.22 (PF10)
- net LTDC_G2: now also U10.42 (PA6)
- net LTDC_G3: now also U10.125 (PG10)
- net LTDC_G4: now also U10.69 (PB10)
- net LTDC_G5: now also U10.70 (PB11)
- net LTDC_G6: now also U10.97 (PC7)
- net LTDC_G7: now also U10.117 (PD3)
- net LTDC_HSYNC: now also U10.96 (PC6)
- net LTDC_R3: now also U10.46 (PB0)
- net LTDC_R4: now also U10.41 (PA5)
- net LTDC_R5: now also U10.101 (PA9)
- net LTDC_R6: now also U10.47 (PB1)
- net LTDC_R7: now also U10.91 (PG6)
- net LTDC_VSYNC: now also U10.40 (PA4)
- net NOR_CLK: now also U10.48 (PB2)
- net NOR_D0: now also U10.20 (PF8)
- net NOR_D1: now also U10.21 (PF9)
- net NOR_D2: now also U10.19 (PF7)
- net NOR_D3: now also U10.18 (PF6)
- net USB_D+: now also U10.104 (PA12)
- net USB_D-: now also U10.103 (PA11)
- net ~{NOR_CS}: now also U10.136 (PB6)
- net PD0 renamed SDRAM_DQ2
- net PD1 renamed SDRAM_DQ3
- net PD10 renamed SDRAM_DQ15
- net PD14 renamed SDRAM_DQ0
- net PD15 renamed SDRAM_DQ1
- net PD8 renamed SDRAM_DQ13
- net PD9 renamed SDRAM_DQ14
- net PE10 renamed SDRAM_DQ7
- net PE11 renamed SDRAM_DQ8
- net PE12 renamed SDRAM_DQ9
- net PE13 renamed SDRAM_DQ10
- net PE14 renamed SDRAM_DQ11
- net PE15 renamed SDRAM_DQ12
- net PE7 renamed SDRAM_DQ4
- net PE8 renamed SDRAM_DQ5
- net PE9 renamed SDRAM_DQ6
- net PF0 renamed SDRAM_ADD0
- net PF1 renamed SDRAM_ADD1
- net PF12 renamed SDRAM_ADD6
- net PF13 renamed SDRAM_ADD7
- net PF14 renamed SDRAM_ADD8
- net PF15 renamed SDRAM_ADD9
- net PF2 renamed SDRAM_ADD2
- net PF3 renamed SDRAM_ADD3
- net PF4 renamed SDRAM_ADD4
- net PF5 renamed SDRAM_ADD5
- net PG0 renamed SDRAM_ADD10
- net PG1 renamed SDRAM_ADD11
Other:
- moved on the sheet: C11, C25, C26, C34, C35, R19, U10

Commit message: Added chroma pixel png
Parts:
- U10: JLCPCB Part # (none) -> C114408
Connections:
- net AUX_SCL: now also U10.81 (PD12)
- net AUX_SDA: now also U10.82 (PD13)
- net BTN0: now also U10.34 (PA0)
- net BTN1: now also U10.35 (PA1)
- net I2S_CK: now also U10.74 (PB13)
- net I2S_SDO: now also U10.29 (PC3_C)
- net I2S_SD_MODE: now also U10.28 (PC2_C)
- net I2S_WS: now also U10.73 (PB12)
- net LCD_TP_INT: now also U10.98 (PC8)
- net LCD_TP_RST: now also U10.137 (PB7)
- net LCD_TP_SCL: now also U10.100 (PA8)
- net LCD_TP_SDA: now also U10.99 (PC9)
- net LED_0: now also U10.127 (PG12)
- net LED_1: now also U10.128 (PG13)
- net SD_CLK: now also U10.27 (PC1)
- net SD_CMD: now also U10.123 (PD7)
- net SD_DAT0: now also U10.75 (PB14)
- net SD_DAT1: now also U10.76 (PB15)
- net SD_DAT2: now also U10.133 (PB3)
- net SD_DAT3: now also U10.134 (PB4)
- net SD_DET: now also U10.135 (PB5)
- net DBG_USART_TX: now reaches U10.119 (PD5)
- net DBG_USART_RX: now reaches U10.122 (PD6)
- net EXT_RX: now reaches U10.124 (PG9)
- net EXT_TX: now reaches U10.129 (PG14)

Commit message: First release H743 version
Parts:
- D7: footprint Package_TO_SOT_SMD:SOT-323_SC-70 -> Package_TO_SOT_SMD:SOT-23
- R22: JLCPCB Part # C25741 -> C60491
Changed lines of the file:
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@@
 			)
 		)
-		(property "JLCPCB Part #" "C25741"
+		(property "JLCPCB Part #" "C60491"
 			(at 308.61 168.91 0)
 			(effects
@@
 			)
 		)
-		(property "Footprint" "Package_TO_SOT_SMD:SOT-323_SC-70"
+		(property "Footprint" "Package_TO_SOT_SMD:SOT-23"
 			(at 116.205 62.865 0)
 			(effects
